Commit message: fkine and ikine test ok

File: model/SA01p.urdf (robot description, URDF)
Before this commit: robot ZQSA01P_Humanoid, 15 links, 14 joints
Joints:
- joint leg_l7_joint: origin xyz=0.06567 0.00592 -0.0495 rpy=0 0 0 -> xyz=0.06567 0.0 -0.0495 rpy=0 0 0
- joint leg_r7_joint: origin xyz=0.06567 -0.00592 -0.0495 rpy=0 0 0 -> xyz=0.06567 0.0 -0.0495 rpy=0 0 0
